File: mikrocontrollerdings.kicad_pcb (KiCad board)
At the start: 2 copper layers, 100.3 x 80 mm, 49 parts, among them CON1 AVR-ISP-6, J1 Conn_Coaxial_Power, J2 MAX232_CONN, J3 EXT, Q1 Q_PNP_CBE, Q2 Q_PNP_CBE, Q3 Q_PNP_CBE, Q4 Q_PNP_CBE, Q5 Q_PNP_CBE, Q6 Q_PNP_CBE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

Commit message: Finish PCB
+ Add GND plane to backside to fix unconnected ground pins
+ Resize +5V track to 1mm
+ Rename LED matrix to correct part
Parts:
- DS1: value TA07-11XWA -> TC07-11XWA
Routing:
- net +5V: track 323.6 -> 326.2 mm, vias 0 -> 1
- added copper zone on F.Cu, net GND
